Commit message: sensores

File: src/orion_description/urdf/orion.urdf.xacro (robot description, xacro)
@@ -10,3 +10,5 @@
     </joint>
     <xacro:include filename="orion_base_gazebo.urdf.xacro"/>
+    <xacro:include filename="sensors/camera.xacro"/>
+    <xacro:include filename="sensors/imus.xacro"/>
 </robot>

File: src/orion_description/urdf/orion_base_gazebo.urdf.xacro (robot description, xacro)
@@ -32,3 +32,30 @@
         </plugin>
     </gazebo>
+    <gazebo>
+        <plugin
+            filename="gz-sim-sensors-system"
+            name="gz::sim::systems::Sensors">
+            <render_engine>ogre2</render_engine>
+        </plugin>
+    </gazebo>
+    <gazebo reference="lidar_link">
+        <sensor name = "lidar" type="gpu_lidar">
+            <topic>scan</topic>
+            <update_rate>10</update_rate>
+            <lidar>
+                <scan>
+                    <horizontal>
+                    <samples>360</samples>
+                    <min_angle>-0.7854</min_angle>
+                    <max_angle>0.7854</max_angle>
+                    </horizontal>
+                </scan>
+                <range>
+                    <min>0.1</min>
+                    <max>10</max>
+                </range>
+            </lidar>
+            <gz_frame_id>lidar_link</gz_frame_id>
+        </sensor>
+    </gazebo>
 </robot>

File: src/orion_description/urdf/sensors/camera.xacro (robot description, xacro)
@@ -22,5 +22,5 @@
         <parent link="base_link"/>
         <child link="camera_link"/>
-        <origin xyz="${(base_lenght+camera_length)/2.0} 0 ${base_height/2}" rpy="0 0 0"/>
+        <origin xyz="${(base_length+camera_length)/2.0} 0 ${base_height/2}" rpy="0 0 0"/>
     </joint>
     <link name="camera_link_optical"></link>
