Commit message: Correction of friction, damping and PID gain of manipulator joint

File: src/orion_description/urdf/orion_base.xacro (robot description, xacro)
@@ -92,4 +92,13 @@
         <origin xyz="${-base_length/3} ${(base_width/2)+(wheel_length/2)} 0" rpy="0 0 0"/>
         <axis xyz="0 1 0"/>
+        <gazebo reference="base_rear_left_wheel">
+            <surface>
+                <friction>
+                    <ode>
+                        <mu>1.0</mu>
+                        <mu2>0.0</mu2> </ode>
+                </friction>
+            </surface>
+        </gazebo>
     </joint>
     <joint name="base_rear_right_wheel" type="continuous">
@@ -98,4 +107,13 @@
         <origin xyz="${-base_length/3} ${(-base_width/2)-(wheel_length/2)} 0" rpy="0 0 0"/>
         <axis xyz="0 1 0"/>
+        <gazebo reference="base_rear_right_wheel">
+            <surface>
+                <friction>
+                    <ode>
+                        <mu>1.0</mu>
+                        <mu2>0.0</mu2> </ode>
+                </friction>
+            </surface>
+        </gazebo>
     </joint>
     <joint name="base_front_left_wheel" type="continuous">
@@ -104,4 +122,13 @@
         <origin xyz="${base_length/3} ${(base_width/2)+(wheel_length/2)} 0" rpy="0 0 0"/>
         <axis xyz="0 1 0"/>
+        <gazebo reference="base_front_left_wheel">
+            <surface>
+                <friction>
+                    <ode>
+                        <mu>1.0</mu>
+                        <mu2>0.0</mu2> </ode>
+                </friction>
+            </surface>
+        </gazebo>
     </joint>
     <joint name="base_front_right_wheel" type="continuous">
@@ -110,4 +137,13 @@
         <origin xyz="${base_length/3} ${(-base_width/2)-(wheel_length/2)} 0" rpy="0 0 0"/>
         <axis xyz="0 1 0"/>
+        <gazebo reference="base_front_right_wheel">
+            <surface>
+                <friction>
+                    <ode>
+                        <mu>1.0</mu>
+                        <mu2>0.0</mu2> </ode>
+                </friction>
+            </surface>
+        </gazebo>
     </joint>
     <joint name="base_support" type="fixed">

File: src/orion_description/urdf/orion_base_gazebo.xacro (robot description, xacro)
@@ -24,10 +24,4 @@
             <joint_name>base_front_left_wheel</joint_name>
             <joint_name>base_front_right_wheel</joint_name>
-            <joint_name>scara_base_first_support_joint</joint_name>
-            <joint_name>first_support_movable_scara_joint</joint_name>
-            <joint_name>arm_joint</joint_name>
-            <joint_name>arm2_base_gripper_joint</joint_name>
-            <joint_name>base_right_gripper_joint</joint_name>
-            <joint_name>base_left_gripper_joint</joint_name>
         </plugin>
     </gazebo>

File: src/orion_description/urdf/orion_manipulator_scara.xacro (robot description, xacro)
@@ -124,5 +124,6 @@
         <origin xyz="0.075 0 0.08" rpy="0 0 0"/>
         <axis xyz="0 0 1"/>
-        <limit lower="-3.14" upper="3.14" effort="10.0" velocity="1.0"/>
+        <limit lower="-3.14" upper="3.14" effort="500.0" velocity="1.0"/>
+        <dynamics friction="20" damping="5" />
     </joint>
     <joint name="support_scara_joint" type="fixed">
@@ -136,5 +137,6 @@
         <origin xyz="0 0 0.075" rpy="0 0 0"/>
         <axis xyz="0 0 1"/>
-        <limit lower="0" upper="0.45" effort="10.0" velocity="1.0"/>
+        <limit lower="0" upper="0.45" effort="300.0" velocity="3.0"/>
+        <dynamics friction="20" damping="5"/>
     </joint>
     <joint name="movable_scara_arm_1_joint" type="fixed">
@@ -148,5 +150,6 @@
         <origin xyz="0.35 0 -0.05" rpy="0 0 0"/>
         <axis xyz="0 0 1"/>
-        <limit lower="-3.14" upper="3.14" effort="10.0" velocity="1.0"/>
+        <limit lower="-3.14" upper="3.14" effort="500.0" velocity="3.0"/>
+        <dynamics friction="15" damping="5" />
     </joint>
     <joint name="arm2_base_gripper_joint" type="revolute">
@@ -155,5 +158,6 @@
         <origin xyz="0.34 0 -0.040" rpy="0 0 0"/>
         <axis xyz="0 0 1"/>
-        <limit lower="-3.14" upper="3.14" effort="10.0" velocity="1.0"/>
+        <limit lower="-3.14" upper="3.14" effort="15.0" velocity="1.0"/>
+        <dynamics friction="5" damping="0.7" />
     </joint>
     <joint name="base_right_gripper_joint" type="prismatic">
@@ -162,5 +166,6 @@
         <origin xyz="0 -0.05 -0.045" rpy="0 0 0"/>
         <axis xyz="0 1 0"/>
-        <limit lower="-0.02" upper="0.02" effort="10.0" velocity="1.0"/>
+        <limit lower="-0.02" upper="0.02" effort="15.0" velocity="1.0"/>
+         <dynamics friction="5.0" damping="0.8"/>
     </joint>
     <joint name="base_left_gripper_joint" type="prismatic">
@@ -169,5 +174,6 @@
         <origin xyz="0 0.05 -0.045" rpy="0 0 0"/>
         <axis xyz="0 1 0"/>
-        <limit lower="-0.02" upper="0.02" effort="10.0" velocity="1.0"/>
+        <limit lower="-0.02" upper="0.02" effort="15.0" velocity="1.0"/>
+        <dynamics friction="5.0" damping="0.8"/>
     </joint>
 </robot>

File: src/orion_description/urdf/orion_manipulator_scara_gazebo.xacro (robot description, xacro)
@@ -7,5 +7,6 @@
             <joint_name>scara_base_first_support_joint</joint_name>
             <topic>/model/orion/joint/scara_arm_joint/0/cmd_pos</topic>
-            <p_gain>5.0</p_gain>
+            <p_gain>50.0</p_gain> <i_gain>25.0</i_gain>  <d_gain>5.0</d_gain>
+            <i_max>15.0</i_max>    <i_min>-15.0</i_min>
         </plugin>
     </gazebo>
@@ -16,5 +17,5 @@
             <joint_name>first_support_movable_scara_joint</joint_name>
             <topic>/model/orion/joint/scara_height_joint/0/cmd_pos</topic>
-            <p_gain>500.0</p_gain> <i_gain>250.0</i_gain>  <d_gain>50.0</d_gain>
+            <p_gain>300.0</p_gain> <i_gain>250.0</i_gain>  <d_gain>90.0</d_gain>
             <i_max>150.0</i_max>    <i_min>-150.0</i_min>
         </plugin>
@@ -26,5 +27,6 @@
             <joint_name>arm_joint</joint_name>
             <topic>/model/orion/joint/scara_arm_joint/1/cmd_pos</topic>
-            <p_gain>5.0</p_gain>
+            <p_gain>100.0</p_gain> <i_gain>50.0</i_gain>  <d_gain>15.0</d_gain>
+            <i_max>15.0</i_max>    <i_min>-15.0</i_min>
         </plugin>
     </gazebo>
@@ -35,4 +37,22 @@
             <joint_name>arm2_base_gripper_joint</joint_name>
             <topic>/model/orion/joint/scara_claw_rotation_joint/0/cmd_pos</topic>
+            <p_gain>3.0</p_gain>
+        </plugin>
+    </gazebo>
+    <gazebo>
+        <plugin
+            filename="gz-sim-joint-position-controller-system"
+            name="gz::sim::systems::JointPositionController">
+            <joint_name>base_right_gripper_joint</joint_name>
+            <topic>/model/orion/joint/scara_gripper/right/cmd_pos</topic>
+            <p_gain>3.0</p_gain>
+        </plugin>
+    </gazebo>
+    <gazebo>
+        <plugin
+            filename="gz-sim-joint-position-controller-system"
+            name="gz::sim::systems::JointPositionController">
+            <joint_name>base_left_gripper_joint</joint_name>
+            <topic>/model/orion/joint/scara_gripper/left/cmd_pos</topic>
             <p_gain>3.0</p_gain>
         </plugin>
