Commit message: Correcao do sensor de altura e adicao de blocos apriltag coloridos

File: src/orion_description/urdf/orion.xacro (robot description, xacro)
@@ -14,5 +14,6 @@
     <xacro:include filename="sensors/imus.xacro"/>
     <xacro:include filename="sensors/lidar.xacro"/>
-    <xacro:include filename="sensors/ultrassonic.xacro"/>
+    <!-- <xacro:include filename="sensors/ultrassonic.xacro"/> -->
     <xacro:include filename="world_sensor_plugins.xacro"/>
+    <xacro:include filename="sensors/distance_laser.xacro"/>
 </robot>

File: src/orion_description/urdf/orion_manipulator_scara.xacro (robot description, xacro)
@@ -135,7 +135,7 @@
         <parent link="first_support_scara_link"/>
         <child link="movable_scara_link"/>
-        <origin xyz="0 0 0.075" rpy="0 0 0"/>
+        <origin xyz="0 0 0.525" rpy="0 0 0"/>
         <axis xyz="0 0 1"/>
-        <limit lower="0" upper="0.45" effort="300.0" velocity="3.0"/>
+        <limit lower="-0.45" upper="0.0" effort="300.0" velocity="3.0"/>
         <dynamics friction="20" damping="5"/>
     </joint>
@@ -164,7 +164,7 @@
         <parent link="base_gripper_link"/>
         <child link="right_gripper_link"/>
-        <origin xyz="0 -0.05 -0.045" rpy="0 0 0"/>
+        <origin xyz="0 -0.07 -0.045" rpy="0 0 0"/>
         <axis xyz="0 1 0"/>
-        <limit lower="-0.02" upper="0.02" effort="100.0" velocity="1.0"/>
+        <limit lower="0" upper="0.04" effort="100.0" velocity="1.0"/>
         <dynamics friction="2.5" damping="0.8"/>
     </joint>
@@ -172,7 +172,7 @@
         <parent link="base_gripper_link"/>
         <child link="left_gripper_link"/>
-        <origin xyz="0 0.05 -0.045" rpy="0 0 0"/>
+        <origin xyz="0 0.07 -0.045" rpy="0 0 0"/>
         <axis xyz="0 1 0"/>
-        <limit lower="-0.02" upper="0.02" effort="100.0" velocity="1.0"/>
+        <limit lower="-0.04" upper="0" effort="100.0" velocity="1.0"/>
         <dynamics friction="2.5" damping="0.8"/>
     </joint>

File: src/orion_description/urdf/sensors/camera.xacro (robot description, xacro)
@@ -66,4 +66,12 @@
                         <stddev>${noise_stddev}</stddev>
                     </noise>
+                    <distortion>
+                        <k1>0.0</k1>
+                        <k2>0.0</k2>
+                        <k3>0.0</k3>
+                        <p1>0.0</p1>
+                        <p2>0.0</p2>
+                        <center>0.5 0.5</center>
+                    </distortion>
                     <optical_frame_id>${name}_link_optical</optical_frame_id>
                     <camera_info_topic>${info_topic}</camera_info_topic>

File: src/orion_description/urdf/sensors/distance_laser.xacro (robot description, xacro)
@@ -1,37 +1,41 @@
 <?xml version="1.0"?>
 <robot xmlns:xacro="http://www.ros.org/wiki/xacro">
-    <xacro:macro name="ultrasonic_module" params="
+    <xacro:macro name="lidar_module" params="
         parent
-        name:=ultrasonic
-        width:=0.02
-        depth:=0.01
-        mass:=0.05
+        name:=distance_sensor
+        radius:=0.02
+        length:=0.01
+        mass:=0.01
         origin_xyz:='0 0 0'
         origin_rpy:='0 0 0'
-        range_min:=0.02
-        range_max:=4.0
+        samples:=360
+        resolution:=1
+        min_angle:=0
+        max_angle:=0
+        range_min:=0.001
+        range_max:=1.0
         range_resolution:=0.01
-        noise_stddev:=0.005
-        update_rate:=20
-        topic:=ultrasonic/range
+        noise_stddev:=0.01
+        update_rate:=10
+        topic:=distance_scan
     ">
         <link name="${name}_frame">
             <visual>
                 <geometry>
-                    <box size="${depth} ${width} ${width}"/>
+                    <cylinder radius="${radius}" length="${length}"/>
                 </geometry>
-                <material name="blue"/>
-                <origin xyz="0 0 0" rpy="0 0 0"/>
+                <material name="yellow"/>
+                <origin xyz="0 0 0" rpy="0 ${pi/2} 0"/>
             </visual>
             <collision>
                 <geometry>
-                    <box size="${depth} ${width} ${width}"/>
+                    <cylinder radius="${radius}" length="${length}"/>
                 </geometry>
-                <origin xyz="0 0 0" rpy="0 0 0"/>
+                <origin xyz="0 0 0" rpy="0 ${pi/2} 0"/>
             </collision>
-            <xacro:box_inertia m="${mass}" x="${depth}" y="${width}" z="${width}"
-                               o_xyz="0 0 0" o_rpy="0 0 0"/>
+            <xacro:cylinder_inertia m="${mass}" r="${radius}" h="${length}"
+                                    o_xyz="0 0 0" o_rpy="0 0 0"/>
         </link>
-        <joint name="${name}_joint" type="fixed">
+        <joint name="${name}_support" type="fixed">
             <parent link="${parent}"/>
             <child link="${name}_frame"/>
@@ -49,8 +53,8 @@
                     <scan>
                         <horizontal>
-                            <samples>1</samples>
-                            <resolution>1</resolution>
-                            <min_angle>0</min_angle>
-                            <max_angle>0</max_angle>
+                            <samples>${samples}</samples>
+                            <resolution>${resolution}</resolution>
+                            <min_angle>${min_angle}</min_angle>
+                            <max_angle>${max_angle}</max_angle>
                         </horizontal>
                     </scan>
@@ -69,8 +73,8 @@
         </gazebo>
     </xacro:macro>
- <!-- <xacro:ultrasonic_module parent="second_support_scara_link"
-    name="ultrasonic_height"
-    origin_xyz="0 0 ${-scara_support_radius/2 + 0.03}"
-    origin_rpy="0 1.5708 0"
-    topic="ultrasonic/height"/> -->
+    <xacro:lidar_module parent="first_support_scara_link"
+                    origin_xyz="0 0 ${scara_support_length}"
+                    origin_rpy="0 ${-pi/2} 0"
+                    min_angle="0"
+                    max_angle="0"/>
 </robot>
