Commit message: Correction of gripper joints overral values

File: src/orion_description/urdf/orion_manipulator_scara.xacro (robot description, xacro)
@@ -158,6 +158,6 @@
         <origin xyz="0.34 0 -0.040" rpy="0 0 0"/>
         <axis xyz="0 0 1"/>
-        <limit lower="-3.14" upper="3.14" effort="15.0" velocity="1.0"/>
-        <dynamics friction="5" damping="0.7" />
+        <limit lower="-3.14" upper="3.14" effort="80.0" velocity="1.0"/>
+        <dynamics friction="5" damping="0.5" />
     </joint>
     <joint name="base_right_gripper_joint" type="prismatic">
@@ -166,6 +166,6 @@
         <origin xyz="0 -0.05 -0.045" rpy="0 0 0"/>
         <axis xyz="0 1 0"/>
-        <limit lower="-0.02" upper="0.02" effort="15.0" velocity="1.0"/>
-         <dynamics friction="5.0" damping="0.8"/>
+        <limit lower="-0.02" upper="0.02" effort="100.0" velocity="1.0"/>
+        <dynamics friction="2.5" damping="0.8"/>
     </joint>
     <joint name="base_left_gripper_joint" type="prismatic">
@@ -174,6 +174,6 @@
         <origin xyz="0 0.05 -0.045" rpy="0 0 0"/>
         <axis xyz="0 1 0"/>
-        <limit lower="-0.02" upper="0.02" effort="15.0" velocity="1.0"/>
-        <dynamics friction="5.0" damping="0.8"/>
+        <limit lower="-0.02" upper="0.02" effort="100.0" velocity="1.0"/>
+        <dynamics friction="2.5" damping="0.8"/>
     </joint>
 </robot>

File: src/orion_description/urdf/orion_manipulator_scara_gazebo.xacro (robot description, xacro)
@@ -37,5 +37,6 @@
             <joint_name>arm2_base_gripper_joint</joint_name>
             <topic>/model/orion/joint/scara_claw_rotation_joint/0/cmd_pos</topic>
-            <p_gain>3.0</p_gain>
+            <p_gain>150.0</p_gain> <i_gain>0.50</i_gain>  <d_gain>15.0</d_gain>
+            <i_max>15.0</i_max>    <i_min>-15.0</i_min>
         </plugin>
     </gazebo>
@@ -46,5 +47,5 @@
             <joint_name>base_right_gripper_joint</joint_name>
             <topic>/model/orion/joint/scara_gripper/right/cmd_pos</topic>
-            <p_gain>3.0</p_gain>
+            <p_gain>500.0</p_gain>
         </plugin>
     </gazebo>
@@ -55,5 +56,5 @@
             <joint_name>base_left_gripper_joint</joint_name>
             <topic>/model/orion/joint/scara_gripper/left/cmd_pos</topic>
-            <p_gain>3.0</p_gain>
+            <p_gain>500.0</p_gain>
         </plugin>
     </gazebo>

Commit message: Some bug fixes

File: src/orion_description/urdf/orion_manipulator_scara.xacro (robot description, xacro)
@@ -137,5 +137,5 @@
         <origin xyz="0 0 0.075" rpy="0 0 0"/>
         <axis xyz="0 0 1"/>
-        <limit lower="0" upper="0.45" effort="300.0" velocity="3.0"/>
+        <limit lower="0" upper="0.45" effort="1000.0" velocity="3.0"/>
         <dynamics friction="20" damping="5"/>
     </joint>

Commit message: Correcao da posicao do sensor de altura

File: src/orion_description/urdf/orion_manipulator_scara.xacro (robot description, xacro)
@@ -135,7 +135,7 @@
         <parent link="first_support_scara_link"/>
         <child link="movable_scara_link"/>
-        <origin xyz="0 0 0.525" rpy="0 0 0"/>
+        <origin xyz="0 0 0.075" rpy="0 0 0"/>
         <axis xyz="0 0 1"/>
-        <limit lower="-0.45" upper="0.0" effort="300.0" velocity="3.0"/>
+        <limit lower="0" upper="0.45" effort="300.0" velocity="3.0"/>
         <dynamics friction="20" damping="5"/>
     </joint>

File: src/orion_description/urdf/orion_manipulator_standalone.xacro (robot description, xacro)
@@ -10,4 +10,5 @@
     <xacro:imu_sensor prefix="arm2" parent="arm_2_link" xyz="0 0 0"/>
     <xacro:imu_sensor prefix="gripper" parent="base_gripper_link" xyz="0 0 0"/>
+    <xacro:include filename="sensors/distance_laser.xacro"/>
     <xacro:include filename="world_sensor_plugins.xacro"/>
 </robot>

File: src/orion_description/urdf/sensors/distance_laser.xacro (robot description, xacro)
@@ -73,7 +73,7 @@
         </gazebo>
     </xacro:macro>
-    <xacro:lidar_module parent="first_support_scara_link"
-                    origin_xyz="0 0 ${scara_support_length}"
-                    origin_rpy="0 ${-pi/2} 0"
+    <xacro:lidar_module parent="second_support_scara_link"
+                    origin_xyz="0 0 0"
+                    origin_rpy="0 ${pi/2} 0"
                     min_angle="0"
                     max_angle="0"/>

Commit message: height pid (height joint error)

File: src/orion_description/urdf/orion_manipulator_scara.xacro (robot description, xacro)
@@ -137,6 +137,6 @@
         <origin xyz="0 0 0.075" rpy="0 0 0"/>
         <axis xyz="0 0 1"/>
-        <limit lower="0" upper="0.45" effort="1000.0" velocity="3.0"/>
-        <dynamics friction="20" damping="5"/>
+        <limit lower="0" upper="0.45" effort="1000.0" velocity="50.0"/>
+        <dynamics friction="0.1" damping="0.5"/>
     </joint>
     <joint name="movable_scara_arm_1_joint" type="fixed">

File: src/orion_description/urdf/orion_manipulator_scara_gazebo.xacro (robot description, xacro)
@@ -7,13 +7,4 @@
             <joint_name>scara_base_first_support_joint</joint_name>
             <topic>/model/orion/joint/scara_arm_joint/0/cmd_pos</topic>
-            <initial_velocity>0</initial_velocity>
-        </plugin>
-    </gazebo>
-    <gazebo>
-        <plugin
-            filename="gz-sim-joint-controller-system"
-            name="gz::sim::systems::JointController">
-            <joint_name>first_support_movable_scara_joint</joint_name>
-            <topic>/model/orion/joint/scara_height_joint/0/cmd_pos</topic>
             <initial_velocity>0</initial_velocity>
         </plugin>

Commit message: Height PID fixed, (It needs to adjust the constants and fix confirmation)

File: src/orion_description/urdf/orion_manipulator_scara.xacro (robot description, xacro)
@@ -137,6 +137,6 @@
         <origin xyz="0 0 0.075" rpy="0 0 0"/>
         <axis xyz="0 0 1"/>
-        <limit lower="0" upper="0.45" effort="1000.0" velocity="50.0"/>
-        <dynamics friction="0.1" damping="0.5"/>
+        <limit lower="0" upper="0.45" effort="1000.0" velocity="0.5"/>
+        <dynamics friction="50" damping="30"/>
     </joint>
     <joint name="movable_scara_arm_1_joint" type="fixed">

File: src/orion_description/urdf/orion_manipulator_scara_gazebo.xacro (robot description, xacro)
@@ -17,4 +17,7 @@
             <topic>/model/orion/joint/scara_height_joint/0/cmd_pos</topic>
             <initial_velocity>0</initial_velocity>
+            <use_force_commands>true</use_force_commands>
+            <p_gain>1</p_gain>
+            <i_gain>0</i_gain>
         </plugin>
     </gazebo>

Commit message: solve_pnp das tags

File: src/orion_description/urdf/orion_manipulator_scara.xacro (robot description, xacro)
@@ -16,5 +16,5 @@
     <xacro:property name="gripper_height" value="0.06"/>
     <xacro:property name="base_scara_mass" value="3.0"/>
-    <xacro:property name="scara_support_mass" value="1.0"/>
+    <xacro:property name="scara_support_mass" value="10.0"/>
     <xacro:property name="arm_mass" value="1.0"/>
     <xacro:property name="base_gripper_mass" value="0.2"/>

File: src/orion_description/urdf/orion_manipulator_standalone.xacro (robot description, xacro)
@@ -1,6 +1,9 @@
 <?xml version="1.0"?>
-<robot name="orion" xmlns:xacro="http://www.ros.org/wiki/xacro">
+<robot name="orion_scara" xmlns:xacro="http://www.ros.org/wiki/xacro">
     <xacro:include filename="common_properties.xacro"/>
     <xacro:include filename="orion_manipulator_scara.xacro"/>
-    <xacro:include filename="orion_manipulador_scara_gazebo.xacro"/>
+    <xacro:include filename="orion_manipulator_scara_gazebo.xacro"/>
+    <xacro:include filename="sensors/camera.xacro"/>
+    <!-- <xacro:include filename="sensors/ultrassonic.xacro"/> -->
+    <xacro:include filename="world_sensor_plugins.xacro"/>
 </robot>
