Commit message: Corrigindo a posicao da camera para ficar na garra

File: src/orion_description/urdf/sensors/camera.xacro (robot description, xacro)
@@ -19,8 +19,8 @@
                            o_xyz="0 0 0" o_rpy="0 0 0"/>
     </link>
-    <joint name="base_camera_joint" type="fixed">
-        <parent link="base_link"/>
+    <joint name="base_gripper_camera_joint" type="fixed">
+        <parent link="base_gripper_link"/>
         <child link="camera_link"/>
-        <origin xyz="${(base_length+camera_length)/2.0} 0 ${base_height/2}" rpy="0 0 0"/>
+        <origin xyz="${(base_gripper_length+camera_height)/2} 0 0" rpy="0 ${pi/2} 0"/>
     </joint>
     <link name="camera_link_optical"></link>

File: src/orion_description/urdf/world_sensor_plugins.xacro (robot description, xacro)
@@ -2,4 +2,5 @@
 <robot name="orion" xmlns:xacro="http://www.ros.org/wiki/xacro">
     <gazebo>
+        <plugin name="gz::sim::systems::Imu" filename="gz-sim-imu-system"/>
         <plugin
             filename="gz-sim-sensors-system"
