Commit message: reajustei a modularizacao

File: orion_description/urdf/sensors/camera.xacro (robot description, xacro)
@@ -4,29 +4,81 @@
     <xacro:property name="camera_width" value="0.1"/>
     <xacro:property name="camera_height" value="0.05"/>
-    <link name="camera_link">
-        <visual>
-            <geometry>
-                <box size="${camera_length} ${camera_width} ${camera_height}"/>
-            </geometry>
-            <material name="grey"/>
-        </visual>
-        <collision>
-            <geometry>
-                <box size="${camera_length} ${camera_width} ${camera_height}"/>
-            </geometry>
-        </collision>
-        <xacro:box_inertia m="0.1" x="${camera_length}" y="${camera_width}" z="${camera_height}"
-                           o_xyz="0 0 0" o_rpy="0 0 0"/>
-    </link>
-    <joint name="base_camera_joint" type="fixed">
-        <parent link="base_link"/>
-        <child link="camera_link"/>
-        <origin xyz="${(base_length+camera_length)/2.0} 0 ${base_height/2}" rpy="0 0 0"/>
-    </joint>
-    <link name="camera_link_optical"></link>
-    <joint name="camera_optical_joint" type="fixed">
-        <origin xyz="0 0 0" rpy="${-pi/2} 0 ${-pi/2}"/>
-        <parent link="camera_link"/>
-        <child link="camera_link_optical"/>
-    </joint>
+    <xacro:macro name="camera_module" params="
+        parent
+        name:=camera
+        length:=0.02
+        width:=0.04
+        height:=0.04
+        mass:=0.1
+        origin_xyz:='0.1 0 0'
+        origin_rpy:='0 ${pi/2} 0'
+        hfov:=1.3962634
+        img_width:=640
+        img_height:=480
+        clip_near:=0.1
+        clip_far:=15
+        noise_stddev:=0.007
+        update_rate:=20
+        topic:=camera/image_raw
+        info_topic:=camera/camera_info
+    ">
+        <link name="${name}_link">
+            <visual>
+                <geometry>
+                    <box size="${length} ${width} ${height}"/>
+                </geometry>
+            </visual>
+            <collision>
+                <geometry>
+                    <box size="${length} ${width} ${height}"/>
+                </geometry>
+            </collision>
+            <xacro:box_inertia m="${mass}" x="${length}" y="${width}" z="${height}"
+                               o_xyz="0 0 0" o_rpy="0 0 0"/>
+        </link>
+        <joint name="${parent}_${name}_joint" type="fixed">
+            <parent link="${parent}"/>
+            <child link="${name}_link"/>
+            <origin xyz="${origin_xyz}" rpy="${origin_rpy}"/>
+        </joint>
+        <link name="${name}_link_optical"/>
+        <joint name="${name}_optical_joint" type="fixed">
+            <parent link="${name}_link"/>
+            <child link="${name}_link_optical"/>
+            <origin xyz="0 0 0" rpy="${-pi/2} 0 ${-pi/2}"/>
+        </joint>
+        <gazebo reference="${name}_link">
+            <sensor name="${name}_sensor" type="camera">
+                <camera>
+                    <horizontal_fov>${hfov}</horizontal_fov>
+                    <image>
+                        <width>${img_width}</width>
+                        <height>${img_height}</height>
+                        <format>R8G8B8</format>
+                    </image>
+                    <clip>
+                        <near>${clip_near}</near>
+                        <far>${clip_far}</far>
+                    </clip>
+                    <noise>
+                        <type>gaussian</type>
+                        <mean>0.0</mean>
+                        <stddev>${noise_stddev}</stddev>
+                    </noise>
+                    <optical_frame_id>${name}_link_optical</optical_frame_id>
+                    <camera_info_topic>${info_topic}</camera_info_topic>
+                </camera>
+                <always_on>1</always_on>
+                <update_rate>${update_rate}</update_rate>
+                <visualize>true</visualize>
+                <topic>${topic}</topic>
+            </sensor>
+        </gazebo>
+    </xacro:macro>
+    <xacro:camera_module parent="base_link"
+                     length="0.01"
+                     width="0.1"
+                     height="0.05"
+                     origin_xyz="${(base_length+0.05)/2.0} 0 0"
+                     origin_rpy="0 ${pi/2} 0"/>
 </robot>

File: orion_description/urdf/sensors/sensors_gazebo.xacro (robot description, xacro)
@@ -37,30 +37,3 @@
         </sensor>
     </gazebo>
-    <gazebo reference="camera_link">
-        <sensor name="camera" type="camera">
-            <camera>
-                <horizontal_fov>1.3962634</horizontal_fov>
-                <image>
-                    <width>640</width>
-                    <height>480</height>
-                    <format>R8G8B8</format>
-                </image>
-                <clip>
-                    <near>0.1</near>
-                    <far>15</far>
-                </clip>
-                <noise>
-                    <type>gaussian</type>
-                    <mean>0.0</mean>
-                    <stddev>0.007</stddev>
-                </noise>
-                <optical_frame_id>camera_link_optical</optical_frame_id>
-                <camera_info_topic>camera/camera_info</camera_info_topic>
-            </camera>
-            <always_on>1</always_on>
-            <update_rate>20</update_rate>
-            <visualize>true</visualize>
-            <topic>camera/image_raw</topic>
-        </sensor>
-    </gazebo>
     </robot>
