Commit message: update

File: orion_description/urdf/orion.xacro (robot description, xacro)
@@ -1,7 +1,7 @@
 <?xml version="1.0"?>
 <robot name="orion" xmlns:xacro="http://www.ros.org/wiki/xacro">
-    <xacro:include filename="common_properties.urdf.xacro"/>
-    <xacro:include filename="orion_base.urdf.xacro"/>
-    <xacro:include filename="orion_manipulator_scara.urdf.xacro"/>
+    <xacro:include filename="common_properties.xacro"/>
+    <xacro:include filename="orion_base.xacro"/>
+    <xacro:include filename="orion_manipulator_scara.xacro"/>
     <joint name="base_scara_joint" type="fixed">
         <parent link="base_link"/>
@@ -9,6 +9,9 @@
         <origin xyz="${(base_length/2) - 0.15} 0 ${base_height}" rpy="0 0 0"/>
     </joint>
-    <xacro:include filename="orion_base_gazebo.urdf.xacro"/>
+    <xacro:include filename="orion_manipulador_scara_gazebo.xacro"/>
+    <xacro:include filename="orion_base_gazebo.xacro"/>
     <xacro:include filename="sensors/camera.xacro"/>
     <xacro:include filename="sensors/imus.xacro"/>
+    <xacro:include filename="sensors/lidar.xacro"/>
+    <xacro:include filename="sensors/sensors_gazebo.xacro"/>
 </robot>

File: orion_description/urdf/orion_base.xacro (robot description, xacro)
@@ -12,5 +12,5 @@
     <xacro:property name="lidar_length" value="0.08"/>
     <xacro:property name="base_mass" value="10.0"/>
-    <xacro:property name="wheel_mass" value="1.5"/>
+    <xacro:property name="wheel_mass" value="5.0"/>
     <xacro:property name="support_lidar_mass" value="0.3"/>
     <xacro:macro name="wheel_link" params="prefix">
@@ -72,13 +72,4 @@
                            o_xyz="${support_length/2} 0 0" o_rpy="0 0 0"/>
     </link>
-    <link name="lidar_link">
-        <visual>
-            <geometry>
-                <cylinder radius="${lidar_radius}" length="${lidar_length}"/>
-            </geometry>
-            <material name="yellow"/>
-            <origin xyz="0 0 0" rpy="0 0 0"/>
-        </visual>
-    </link>
     --------------------------------------------------
     <joint name="base_joint" type="fixed">
@@ -116,8 +107,3 @@
         <origin xyz="${(base_length/2)} 0 ${support_height/2}" rpy="0 0 0"/>
     </joint>
-    <joint name="lidar_support" type="fixed">
-        <parent link="support_link"/>
-        <child link="lidar_link"/>
-        <origin xyz="${support_length/2} 0 ${(support_height/2)+(lidar_length/2)}" rpy="0 0 0"/>
-    </joint>
 </robot>

File: orion_description/urdf/orion_manipulator_scara.xacro (robot description, xacro)
@@ -125,4 +125,5 @@
         <axis xyz="0 0 1"/>
         <limit lower="-3.14" upper="3.14" effort="10.0" velocity="1.0"/>
+        <dynamics friction="0.8" damping="0.3" />
     </joint>
     <joint name="support_scara_joint" type="fixed">
@@ -136,5 +137,5 @@
         <origin xyz="0 0 0.075" rpy="0 0 0"/>
         <axis xyz="0 0 1"/>
-        <limit lower="0" upper="0.45" effort="10.0" velocity="1.0"/>
+        <limit lower="0" upper="0.45" effort="500.0" velocity="1.0"/>
     </joint>
     <joint name="movable_scara_arm_1_joint" type="fixed">
@@ -149,4 +150,5 @@
         <axis xyz="0 0 1"/>
         <limit lower="-3.14" upper="3.14" effort="10.0" velocity="1.0"/>
+        <dynamics friction="0.8" damping="0.3" />
     </joint>
     <joint name="arm2_base_gripper_joint" type="revolute">
@@ -156,4 +158,5 @@
         <axis xyz="0 0 1"/>
         <limit lower="-3.14" upper="3.14" effort="10.0" velocity="1.0"/>
+        <dynamics friction="0.3" damping="0.3" />
     </joint>
     <joint name="base_right_gripper_joint" type="prismatic">

File: orion_description/urdf/sensors/camera.xacro (robot description, xacro)
@@ -30,30 +30,3 @@
         <child link="camera_link_optical"/>
     </joint>
-    <gazebo reference="camera_link">
-        <sensor name="camera" type="camera">
-            <camera>
-                <horizontal_fov>1.3962634</horizontal_fov>
-                <image>
-                    <width>640</width>
-                    <height>480</height>
-                    <format>R8G8B8</format>
-                </image>
-                <clip>
-                    <near>0.1</near>
-                    <far>15</far>
-                </clip>
-                <noise>
-                    <type>gaussian</type>
-                    <mean>0.0</mean>
-                    <stddev>0.007</stddev>
-                </noise>
-                <optical_frame_id>camera_link_optical</optical_frame_id>
-                <camera_info_topic>camera/camera_info</camera_info_topic>
-            </camera>
-            <always_on>1</always_on>
-            <update_rate>20</update_rate>
-            <visualize>true</visualize>
-            <topic>camera/image_raw</topic>
-        </sensor>
-    </gazebo>
 </robot>

Commit message: modularizacao

File: orion_description/urdf/orion.xacro (robot description, xacro)
@@ -1,4 +1,11 @@
 <?xml version="1.0"?>
 <robot name="orion" xmlns:xacro="http://www.ros.org/wiki/xacro">
+        <gazebo>
+            <plugin
+                filename="gz-sim-sensors-system"
+                name="gz::sim::systems::Sensors">
+                <render_engine>ogre2</render_engine>
+            </plugin>
+        </gazebo>
     <xacro:include filename="common_properties.xacro"/>
     <xacro:include filename="orion_base.xacro"/>
@@ -14,4 +21,3 @@
     <xacro:include filename="sensors/imus.xacro"/>
     <xacro:include filename="sensors/lidar.xacro"/>
-    <xacro:include filename="sensors/sensors_gazebo.xacro"/>
 </robot>

File: orion_description/urdf/sensors/camera.xacro (robot description, xacro)
@@ -38,5 +38,5 @@
         </link>
         <joint name="${parent}_${name}_joint" type="fixed">
-            <parent link="${parent}"/>
+            <parent link="${parent}_link"/>
             <child link="${name}_link"/>
             <origin xyz="${origin_xyz}" rpy="${origin_rpy}"/>
@@ -76,9 +76,9 @@
         </gazebo>
     </xacro:macro>
-    <xacro:camera_module parent="base_link"
+    <xacro:camera_module parent="base_gripper"
                      length="0.01"
                      width="0.1"
                      height="0.05"
-                     origin_xyz="${(base_length+0.05)/2.0} 0 0"
+                     origin_xyz="${(base_gripper_length+0.05)/2.0} 0 0"
                      origin_rpy="0 ${pi/2} 0"/>
 </robot>

File: orion_description/urdf/sensors/lidar.xacro (robot description, xacro)
@@ -1,25 +1,82 @@
 <?xml version="1.0"?>
 <robot xmlns:xacro="http://www.ros.org/wiki/xacro">
-<link name="laser_frame">
-        <visual>
-            <geometry>
-                <cylinder radius="${lidar_radius}" length="${lidar_length}"/>
-            </geometry>
-            <material name="yellow"/>
-            <origin xyz="0 0 0" rpy="0 0 0"/>
-        </visual>
-        <collision>
-            <geometry>
-                <cylinder radius="${lidar_radius}" length="${lidar_length}"/>
-            </geometry>
-            <origin xyz="0 0 0" rpy="0 0 0"/>
-        </collision>
-        <xacro:cylinder_inertia m="0.2" r="${lidar_radius}" h="${lidar_length}"
+    <xacro:macro name="lidar_module" params="
+        parent
+        name:=laser
+        radius:=0.05
+        length:=0.04
+        mass:=0.2
+        origin_xyz:='0 0 0'
+        origin_rpy:='0 0 0'
+        samples:=360
+        resolution:=1
+        min_angle:=-3.14159
+        max_angle:=3.14159
+        range_min:=0.15
+        range_max:=10.0
+        range_resolution:=0.01
+        noise_stddev:=0.01
+        update_rate:=10
+        topic:=scan
+    ">
+        <link name="${name}_frame">
+            <visual>
+                <geometry>
+                    <cylinder radius="${radius}" length="${length}"/>
+                </geometry>
+                <material name="yellow"/>
+                <origin xyz="0 0 0" rpy="0 0 0"/>
+            </visual>
+            <collision>
+                <geometry>
+                    <cylinder radius="${radius}" length="${length}"/>
+                </geometry>
+                <origin xyz="0 0 0" rpy="0 0 0"/>
+            </collision>
+            <xacro:cylinder_inertia m="${mass}" r="${radius}" h="${length}"
                                     o_xyz="0 0 0" o_rpy="0 0 0"/>
-    </link>
-    <joint name="lidar_support" type="fixed">
-        <parent link="support_link"/>
-        <child link="laser_frame"/>
-        <origin xyz="${support_length/2} 0 ${(support_height/2)+(lidar_length/2)}" rpy="0 0 0"/>
-    </joint>
+        </link>
+        <joint name="${name}_support" type="fixed">
+            <parent link="${parent}"/>
+            <child link="${name}_frame"/>
+            <origin xyz="${origin_xyz}" rpy="${origin_rpy}"/>
+        </joint>
+        <gazebo reference="${name}_frame">
+            <sensor name="${name}" type="gpu_lidar">
+                <pose>0 0 0 0 0 0</pose>
+                <always_on>true</always_on>
+                <visualize>true</visualize>
+                <update_rate>${update_rate}</update_rate>
+                <topic>${topic}</topic>
+                <gz_frame_id>${name}_frame</gz_frame_id>
+                <lidar>
+                    <scan>
+                        <horizontal>
+                            <samples>${samples}</samples>
+                            <resolution>${resolution}</resolution>
+                            <min_angle>${min_angle}</min_angle>
+                            <max_angle>${max_angle}</max_angle>
+                        </horizontal>
+                    </scan>
+                    <range>
+                        <min>${range_min}</min>
+                        <max>${range_max}</max>
+                        <resolution>${range_resolution}</resolution>
+                    </range>
+                    <noise>
+                        <type>gaussian</type>
+                        <mean>0.0</mean>
+                        <stddev>${noise_stddev}</stddev>
+                    </noise>
+                </lidar>
+            </sensor>
+        </gazebo>
+    </xacro:macro>
+    <xacro:lidar_module parent="support_link"
+                    radius="${lidar_radius}"
+                    length="${lidar_length}"
+                    origin_xyz="${support_length/2} 0 ${(support_height/2)+(lidar_length/2)}"
+                    origin_rpy="0 0 0"
+                    min_angle="${-pi/2}"
+                    max_angle="${pi/2}"/>
 </robot>
